File: bbq10breakout.sch (KiCad schematic (older format))
At the start: 4 parts, among them J1 Conn_01x08, J2 Conn_01x08, U1 BBQ10KBD

Commit message: Added gerbers and updated the files to latest nightly
Parts:
- C1: symbol device:C_Small -> Device:C_Small
- J1, J2: symbol Connector:Conn_01x08 -> Connector_Generic:Conn_01x08
Connections:
- wire segments 38 -> 40
Changed lines of the file:
@@
 EESchema Schematic File Version 4
+LIBS:bbq10breakout-cache
 EELAYER 26 0
 EELAYER END
@@
 $EndComp
 Wire Wire Line
-	5300 2200 5400 2200
+	5300 2200 5350 2200
 Wire Wire Line
 	5350 2200 5350 2150
@@
 	5400 3300 5350 3300
 Wire Wire Line
-	5350 3300 5350 3450
+	5350 3300 5350 3400
 Wire Wire Line
 	5350 3400 5400 3400
@@
 $EndComp
 $Comp
-L device:C_Small C1
+L Device:C_Small C1
 U 1 1 5A384436
 P 5200 2200
@@
 $EndComp
 $Comp
-L Connector:Conn_01x08 J1
+L Connector_Generic:Conn_01x08 J1
 U 1 1 5A38AC19
 P 8300 1550
@@
 $EndComp
 $Comp
-L Connector:Conn_01x08 J2
+L Connector_Generic:Conn_01x08 J2
 U 1 1 5A38BC0E
 P 9400 1550
@@
 	9600 1250 9650 1250
 NoConn ~ 9600 1950
+Wire Wire Line
+	5350 3400 5350 3450
+Wire Wire Line
+	5350 2200 5400 2200
 $EndSCHEMATC
